File: GD32F505_FOC.kicad_sch (KiCad schematic)
At the start: 52 parts, among them Q1 IRFB4110PBF, Q10 IRFB4110PBF, Q11 IRFB4110PBF, Q12 IRFB4110PBF, Q2 IRFB4110PBF, Q3 IRFB4110PBF, Q4 IRFB4110PBF, Q5 IRFB4110PBF, Q6 IRFB4110PBF, Q7 IRFB4110PBF, Q8 IRFB4110PBF, Q9 IRFB4110PBF, U1 GD32F505VGT7, U10 TLV9062IDGKT, U11 TPS54560DDAR, U12 78M05, U13 LD1117AG-3.3V-A, U2 DRV8300NPWR, U3 DRV8300NPWR, U8 TLV9062IDGKT, U9 TLV9062IDGKT

Commit message: sch_v0
Parts:
- added CN1: XT30PW-M, kicad_api_lib:XT30PW-M, symbol XT30PW-M:XT30PW-M
Changed lines of the file:
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@@
+	)
+	(symbol
+		(lib_id "XT30PW-M:XT30PW-M")
+		(at 219.71 96.52 0)
+		(unit 1)
+		(body_style 1)
+		(exclude_from_sim no)
+		(in_bom yes)
+		(on_board yes)
+		(in_pos_files yes)
+		(dnp no)
+		(fields_autoplaced yes)
+		(property "Reference" "CN1"
+			(at 219.71 90.17 0)
+			(show_name no)
+			(do_not_autoplace no)
+			(effects
+				(font
+					(size 1.27 1.27)
+				)
+			)
+		)
+		(property "Value" "XT30PW-M"
+			(at 219.71 92.71 0)
+			(show_name no)
+			(do_not_autoplace no)
+			(effects
+				(font
+					(size 1.27 1.27)
+				)
+			)
+		)
+		(property "Footprint" "kicad_api_lib:XT30PW-M"
+			(at 219.71 92.71 0)
+			(hide yes)
+			(show_name no)
+			(do_not_autoplace no)
+			(effects
+				(font
+					(size 1.27 1.27)
+				)
+			)
+		)
+		(property "Datasheet" "http://file.elecfans.com/web1/M00/DA/CE/pIYBAGAADk-ANpM1ARYS5bgBxnI084.pdf"
+			(at 219.71 92.71 0)
+			(hide yes)
+			(show_name no)
+			(do_not_autoplace no)
+			(effects
+				(font
+					(size 1.27 1.27)
+				)
+			)
+		)
+		(property "Description" "Socket,DCsupply,XT30,male,PIN:2"
+			(at 219.71 92.71 0)
+			(hide yes)
+			(show_name no)
+			(do_not_autoplace no)
+			(effects
+				(font
+					(size 1.27 1.27)
+				)
+			)
+		)
+		(property "MPN" "XT30PW-M"
+			(at 219.71 96.52 0)
+			(hide yes)
+			(show_name no)
+			(do_not_autoplace no)
+			(effects
+				(font
+					(size 1.27 1.27)
+				)
+			)
+		)
+		(property "Manufacturer" "Amass"
+			(at 219.71 96.52 0)
+			(hide yes)
+			(show_name no)
+			(do_not_autoplace no)
+			(effects
+				(font
+					(size 1.27 1.27)
+				)
+			)
+		)
+		(property "contact_plating" "镀金"
+			(at 219.71 96.52 0)
+			(hide yes)
+			(show_name no)
+			(do_not_autoplace no)
+			(effects
+				(font
+					(size 1.27 1.27)
+				)
+			)
+		)
+		(property "huaqiu_pn" "G4619089"
+			(at 219.71 96.52 0)
+			(hide yes)
+			(show_name no)
+			(do_not_autoplace no)
+			(effects
+				(font
+					(size 1.27 1.27)
+				)
+			)
+		)
+		(property "lead_free" "Yes"
+			(at 219.71 96.52 0)
+			(hide yes)
+			(show_name no)
+			(do_not_autoplace no)
+			(effects
+				(font
+					(size 1.27 1.27)
+				)
+			)
+		)
+		(property "mount" "DIP"
+			(at 219.71 96.52 0)
+			(hide yes)
+			(show_name no)
+			(do_not_autoplace no)
+			(effects
+				(font
+					(size 1.27 1.27)
+				)
+			)
+		)
+		(property "package" "CONN_13.3X14.9MM_TM"
+			(at 219.71 96.52 0)
+			(hide yes)
+			(show_name no)
+			(do_not_autoplace no)
+			(effects
+				(font
+					(size 1.27 1.27)
+				)
+			)
+		)
+		(property "packaging" "500pcs"
+			(at 219.71 96.52 0)
+			(hide yes)
+			(show_name no)
+			(do_not_autoplace no)
+			(effects
+				(font
+					(size 1.27 1.27)
+				)
+			)
+		)
+		(property "pins" "2"
+			(at 219.71 96.52 0)
+			(hide yes)
+			(show_name no)
+			(do_not_autoplace no)
+			(effects
+				(font
+					(size 1.27 1.27)
+				)
+			)
+		)
+		(pin "3"
+		)
+		(pin "4"
+		)
+		(pin "1"
+		)
+		(pin "2"
+		)
+		(instances
+			(project "GD32F505_FOC"
+				(path "/fde07a63-2c29-4735-b4b4-3708b0afb980"
+					(reference "CN1")
+					(unit 1)
+				)
+			)
+		)
 	)
 	(symbol
